File: Hardware/single-layer-modules/single-layer-modules.kicad_sch (KiCad schematic)
At the start: 0 parts

Commit message: Refactor code structure for improved readability and maintainability
Parts:
- added C1: C_Polarized, Capacitor_THT:CP_Radial_D17.0mm_P7.50mm, symbol Device:C_Polarized
- added J1: Blue Pill - 1, Connector_PinHeader_2.54mm:PinHeader_1x20_P2.54mm_Vertical, symbol Connector:Conn_01x20_Socket
- added J2: Blue Pill - 2, Connector_PinHeader_2.54mm:PinHeader_1x20_P2.54mm_Vertical, symbol Connector:Conn_01x20_Socket
- added J3: SIM800L, Connector_PinSocket_2.54mm:PinSocket_1x07_P2.54mm_Vertical, symbol Connector:Conn_01x07_Socket
- added J4: DS18B20, Connector_PinSocket_2.54mm:PinSocket_1x03_P2.54mm_Vertical, symbol Connector:Conn_01x03_Socket
- added J5: DHT11, Connector_PinSocket_2.54mm:PinSocket_1x03_P2.54mm_Vertical, symbol Connector:Conn_01x03_Socket
- added J6: FC-28, Connector_PinSocket_2.54mm:PinSocket_1x03_P2.54mm_Vertical, symbol Connector:Conn_01x03_Socket
- added J7: MQ-02, Connector_PinSocket_2.54mm:PinSocket_1x03_P2.54mm_Vertical, symbol Connector:Conn_01x03_Socket
- added J8: FC-37, Connector_PinSocket_2.54mm:PinSocket_1x03_P2.54mm_Vertical, symbol Connector:Conn_01x03_Socket
Connections:
- new net +3.3V: J1.1 (Pin_1), J2.18 (Pin_18)
- new net +5V: J1.3 (Pin_3)
- new net GND: J1.2 (Pin_2), J2.19 (Pin_19), J2.20 (Pin_20)
- new net PA_0: J2.5 (Pin_5)
- new net PA_1: J2.6 (Pin_6)
- new net PA_2: J2.7 (Pin_7)
- new net PA_3: J2.8 (Pin_8)
- new net PA_4: J2.9 (Pin_9)
- new net PA_5: J2.10 (Pin_10)
- new net PA_6: J2.11 (Pin_11)
- new net PA_7: J2.12 (Pin_12)
- new net PB_0: J2.13 (Pin_13)
- new net PB_1: J1.20 (Pin_20), J2.14 (Pin_14)
- new net PB_10: J2.15 (Pin_15)
- new net PB_11: J2.16 (Pin_16)
- new net PC_13: J2.2 (Pin_2)
- new net PC_14: J2.3 (Pin_3)
- new net PC_15: J2.4 (Pin_4)
- new net RESET: J2.17 (Pin_17)
- new net VCC_RTC: J2.1 (Pin_1)
