File: Hardware/single-layer-modules/single-layer-modules.kicad_sch (KiCad schematic)
At the start: 19 parts, among them J1 Blue Pill - 1, J2 Blue Pill - 2, J3 SIM800L, J4 DS18B20, J5 DHT11, J6 FC-28, J7 MQ-02, Q1 FDS9435A, Q2 2N3904, SW1 SW_DIP_x05

Commit message: Add New PCB
Parts:
- removed Q1: FDS9435A, Package_SO:SOIC-8_3.9x4.9mm_P1.27mm, symbol Transistor_FET:FDS9435A
- added C2, C3: C_Polarized, Capacitor_THT:CP_Radial_D17.0mm_P7.50mm, symbol Device:C_Polarized
- added D1, D2: 1N4448, Diode_THT:D_DO-35_SOD27_P7.62mm_Horizontal, symbol Diode:1N4448
- added J10, J11, J8, J9: Conn_01x01_Pin, Connector_PinSocket_2.54mm:PinSocket_1x01_P2.54mm_Vertical, symbol Connector:Conn_01x01_Pin
- added J12: Conn_01x02_Socket, Connector_AMASS:AMASS_XT30UPB-M_1x02_P5.0mm_Vertical, symbol Connector:Conn_01x02_Socket
- added JP1: SolderJumper_3_Bridged12, Connector_JST:JST_PH_S3B-PH-K_1x03_P2.00mm_Horizontal, symbol Jumper:SolderJumper_3_Bridged12
- added Q1: IRF4905, Package_TO_SOT_THT:TO-220-3_Vertical, symbol Transistor_FET:IRF4905
- added R10, R11, R12, R13, R14, R15, R16, R17, R18, R19, R20, R21, R22, R23, R24, R9: R, Resistor_THT:R_Axial_DIN0411_L9.9mm_D3.6mm_P15.24mm_Horizontal, symbol Device:R
- added U1, U2: LM358, Package_DIP:DIP-8_W7.62mm_LongPads, symbol Amplifier_Operational:LM358
Connections:
- net +3.3V: now also JP1.3 (B)
- net +5V: now also J10.1 (Pin_1), Q1.2 (D), R24.1, R24.2
- net GND: now also C3.2, J11.1 (Pin_1), J12.2 (Pin_2), J9.1 (Pin_1), R11.1, R18.2, R20.1, U2.4 (V-)
- net PA_2: now also R21.2; no longer J3.4 (Pin_4)
- net PA_3: now also R22.2; no longer J3.5 (Pin_5)
- net PA_6: now also R19.1, R20.2
- net PB_3: now also R23.2
- net VCC_5V: now also JP1.1 (A), Q1.3 (S); no longer J3.3 (Pin_3)
- net at R8.1: now also Q1.1 (G)
- net at R7.2: now also R23.1
- new net: D2.2 (A), U2.1
- new net: R14.1, U2.2 (-)
- new net: R15.1, U2.3 (+)
- new net: J3.4 (Pin_4), R21.1
- new net: C2.2, C3.1
- new net: D2.1 (K), R10.1, R11.2
- new net: R15.2, R16.2, R18.1
- new net: J3.5 (Pin_5), R22.1
- new net: R13.2, R16.1, R17.2
- new net: R12.2, R14.2
- new net: R12.1, U1.3 (+)
- new net: R13.1, U1.2 (-)
- new net: D1.1 (K), R10.2, R9.1
- new net: D1.2 (A), U1.1
- new net: U1.4 (V-), U2.8 (V+)
- new net SIM800L: J3.3 (Pin_3), JP1.2 (C)
- new net SOLAR_REG_IN: C2.1, J12.1 (Pin_1), R17.1, R19.2, U1.8 (V+)
- new net VCC_IN: J8.1 (Pin_1), R9.2
