File: Hardware/single-layer-modules/_autosave-single-layer-modules.kicad_pcb (KiCad board)
At the start: 2 copper layers, 150.5 x 90.5 mm, 20 parts, among them J1 Blue Pill - 1, J2 Blue Pill - 2, J3 SIM800L, J4 DS18B20, J5 DHT11, J6 FC-28, J7 MQ-02, J8 FC-37, Q1 FDS9435A, Q2 2N3904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

Commit message: Add autosave and backup files for PCB project
Added KiCad autosave and backup files for the single-layer-modules project, including .kicad_pcb, .kicad_sch, and backup zip archives. Updated main PCB and schematic files with recent changes. Lock files for autosave and schematic were also added.
Parts:
- moved J7 8.75 mm to (166.4, 49.4)
- moved J8 8.75 mm to (171.0, 49.4)
Changed lines of the file:
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@@
 	(footprint "Connector_PinSocket_2.54mm:PinSocket_1x03_P2.54mm_Vertical"
 		(layer "F.Cu")
-		(at 175.15 49.46)
+		(at 166.4 49.42)
 		(descr "Through hole straight socket strip, 1x03, 2.54mm pitch, single row (from Kicad 4.0.7), script generated")
 		(tags "Through hole socket strip THT 1x03 2.54mm single row")
@@
 	(footprint "Connector_PinSocket_2.54mm:PinSocket_1x03_P2.54mm_Vertical"
 		(layer "F.Cu")
-		(at 179.75 49.46)
+		(at 171 49.42)
 		(descr "Through hole straight socket strip, 1x03, 2.54mm pitch, single row (from Kicad 4.0.7), script generated")
 		(tags "Through hole socket strip THT 1x03 2.54mm single row")
